Commit message: Add files via upload

File: refer 2/Drawing Arm Solidworks/Draw_armV3.urdf (robot description, URDF)
Before this commit: robot Draw_armV3, 6 links, 5 joints
Joints:
- joint jnt2: limit lower=-3.14 upper=3.14 effort=0 velocity=0 -> lower=-1.571 upper=1.571 effort=0 velocity=0
- joint jnt3: limit lower=-3.14 upper=3.14 effort=0 velocity=0 -> lower=-1.571 upper=1.571 effort=0 velocity=0
- joint jnt4: limit lower=-3.14 upper=3.14 effort=0 velocity=0 -> lower=-1.571 upper=1.571 effort=0 velocity=0
