Commit message: Add files via upload

File: refer 2/Drawing Arm Solidworks/Draw_armV6.urdf (robot description, URDF)
Before this commit: robot Draw_armV6, 5 links, 4 joints
Links:
- link Plate: geometry collision mesh filename=Plate.STL; visual mesh filename=Plate.STL
- link body1: geometry collision mesh filename=body1.STL; visual mesh filename=body1.STL
- link body2: geometry collision mesh filename=body2.STL; visual mesh filename=body2.STL
- link body3: geometry collision mesh filename=body3.STL; visual mesh filename=body3.STL
- link body4: geometry collision mesh filename=body4.STL; visual mesh filename=body4.STL
Joints:
- joint jnt2: limit lower=-2.356 upper=3.14 effort=0 velocity=0 -> lower=-1.5708 upper=1.5708 effort=0 velocity=0
- joint jnt3: limit lower=-3.14 upper=3.14 effort=0 velocity=0 -> lower=-2.094 upper=2.094 effort=0 velocity=0
