Commit message: FINAL APP

File: Draw_armV6.urdf (robot description, URDF)
Before this commit: robot Draw_armV6, 5 links, 4 joints
Links:
- link Plate: geometry collision mesh filename=package://Draw_armV6/meshes/Plate.STL; visual mesh filename=package://Draw_armV6/meshes/Plate.STL
- link body1: geometry collision mesh filename=package://Draw_armV6/meshes/body1.STL; visual mesh filename=package://Draw_armV6/meshes/body1.STL
- link body2: geometry collision mesh filename=package://Draw_armV6/meshes/body2.STL; visual mesh filename=package://Draw_armV6/meshes/body2.STL
- link body3: geometry collision mesh filename=package://Draw_armV6/meshes/body3.STL; visual mesh filename=package://Draw_armV6/meshes/body3.STL
- link body4: geometry collision mesh filename=package://Draw_armV6/meshes/body4.STL; visual mesh filename=package://Draw_armV6/meshes/body4.STL
Joints:
- joint jnt2: limit lower=-1.5708 upper=1.5708 effort=0 velocity=0 -> lower=-2.356 upper=3.14 effort=0 velocity=0
- joint jnt3: limit lower=-2.094 upper=2.094 effort=0 velocity=0 -> lower=-3.14 upper=3.14 effort=0 velocity=0
